File: PCB_MF_PicoMicro.kicad_sch (KiCad schematic)
At the start: 10 parts, among them J1 Conn_01x12, J2 Conn_01x12, J7 Conn_01x02_Pin, J8 Conn_01x02_Pin

Commit message: better positioning of parts
Parts:
- R11, R12: value 100 -> 50
Changed lines of the file:
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@@
 			)
 		)
-		(property "Value" "100"
+		(property "Value" "50"
 			(at 140.208 111.76 90)
 			(effects
@@
 			)
 		)
-		(property "Value" "100"
+		(property "Value" "50"
 			(at 202.946 111.76 90)
 			(effects
