File: RP2040.kicad_sch (KiCad schematic)
At the start: 35 parts, among them J3 USB_C_Receptacle_USB2.0_16P, SW1 SW_Push, U1 RP2040, U2 AMS1117-3.3, U4 W25Q16JVSS, Y1 X322512MSB4SI

Commit message: route both additional resistors
Other:
- moved on the sheet: C1, C10, C11, C12, C13, C14, C15, C16, C17, C18, C19, C2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

Commit message: update production files
Parts:
- C11, C12, C13, C14, C15, C6, C9: value 100n -> 100nF
Changed lines of the file:
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@@
 			)
 		)
-		(property "Value" "100n"
+		(property "Value" "100nF"
 			(at 223.901 30.353 0)
 			(effects
@@
 			)
 		)
-		(property "Value" "100n"
+		(property "Value" "100nF"
 			(at 211.836 30.988 0)
 			(effects
@@
 			)
 		)
-		(property "Value" "100n"
+		(property "Value" "100nF"
 			(at 157.861 31.623 0)
 			(effects
@@
 			)
 		)
-		(property "Value" "100n"
+		(property "Value" "100nF"
 			(at 258.191 30.353 0)
 			(effects
@@
 			)
 		)
-		(property "Value" "100n"
+		(property "Value" "100nF"
 			(at 246.761 30.353 0)
 			(effects
@@
 			)
 		)
-		(property "Value" "100n"
+		(property "Value" "100nF"
 			(at 269.621 30.353 0)
 			(effects
@@
 			)
 		)
-		(property "Value" "100n"
+		(property "Value" "100nF"
 			(at 235.331 30.353 0)
 			(effects

Commit message: update production files
Parts:
- U1: value RP2040 -> RP2350A
Changed lines of the file:
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@@
 			)
 		)
-		(property "Value" "RP2040"
+		(property "Value" "RP2350A"
 			(at 228.6 154.94 0)
 			(effects
